File: hardware/FLC100_shield/shield_v2.0/FLC100_shield_v2.0.sch (EAGLE design)
At the start: 68 parts, among them IC1 TSR 1-2450, IC4 MCP1640SOT23-6-HAND, J1 RJ11-6PTH, Q1 2N7000, Q2 2N7000, Q3 2N7000, Q4 2N7000, Q5 2N7000, Q6 2N7000, Q7 2N7000, Q8 2N7000, Q9 2N7000, X1 RJ45, X2 CLOUD SENSOR, X4 HUMIDITY, X5 SMA

Commit message: Development of new FLC100 shield.
Parts:
- added C4: 100n, SparkFun:CAPPTH
Connections:
- net +5V: no longer X4.1
- net GND: now also C4.2
- net IOREF: now also X4.1
- net N$22: now also C4.1
Other:
- note added: "No level-shifting so maximum pull-up voltage should be IOREF."
- moved on the sheet: C2, C3
Changed lines of the file:
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@@
 <part name="R20" library="SteveMarple" deviceset="RESISTOR" device="" value="10k"/>
 <part name="P+6" library="supply1" deviceset="+5V" device=""/>
-<part name="P+11" library="supply1" deviceset="+5V" device=""/>
 <part name="C3" library="SparkFun" deviceset="CAP_POL" device="PTH2" value="4u7 25V"/>
 <part name="GND12" library="supply1" deviceset="GND" device=""/>
@@
 <part name="GND14" library="supply1" deviceset="GND" device=""/>
 <part name="JP1" library="SparkFun" deviceset="JUMPER-3" device="PTH" value="ISP VCC"/>
+<part name="C4" library="SparkFun" deviceset="CAP" device="PTH" value="100n"/>
+<part name="GND21" library="supply1" deviceset="GND" device=""/>
 </parts>
 <sheets>
@@
 <text x="317.5" y="200.66" size="1.778" layer="91">Voltage selection for battery or
 power-over-ethernet operation.</text>
+<text x="317.5" y="30.48" size="1.778" layer="91">No level-shifting so maximum pull-up
+voltage should be IOREF.</text>
 </plain>
 <instances>
@@
 <instance part="U$40" gate="G$1" x="238.76" y="-66.04" rot="R180"/>
 <instance part="JP13" gate="A" x="137.16" y="215.9"/>
-<instance part="C2" gate="G$1" x="223.52" y="33.02"/>
-<instance part="GND9" gate="1" x="223.52" y="25.4"/>
+<instance part="C2" gate="G$1" x="203.2" y="33.02"/>
+<instance part="GND9" gate="1" x="203.2" y="25.4"/>
 <instance part="+3V6" gate="G$1" x="261.62" y="45.72"/>
-<instance part="GND10" gate="1" x="264.16" y="25.4"/>
+<instance part="GND10" gate="1" x="264.16" y="20.32"/>
 <instance part="U$5" gate="G$1" x="284.48" y="33.02"/>
 <instance part="R19" gate="G$1" x="284.48" y="48.26" rot="R90"/>
 <instance part="R20" gate="G$1" x="292.1" y="48.26" rot="R90"/>
 <instance part="P+6" gate="1" x="281.94" y="137.16"/>
-<instance part="P+11" gate="1" x="299.72" y="30.48" rot="R270"/>
-<instance part="C3" gate="G$1" x="233.68" y="33.02"/>
-<instance part="GND12" gate="1" x="233.68" y="25.4"/>
-<instance part="P+12" gate="1" x="233.68" y="40.64"/>
+<instance part="C3" gate="G$1" x="213.36" y="33.02"/>
+<instance part="GND12" gate="1" x="213.36" y="25.4"/>
+<instance part="P+12" gate="1" x="213.36" y="40.64"/>
 <instance part="+3V7" gate="G$1" x="231.14" y="-96.52"/>
 <instance part="GND13" gate="1" x="231.14" y="-129.54"/>
@@
 <instance part="GND14" gate="1" x="205.74" y="-111.76"/>
 <instance part="JP1" gate="G$1" x="309.88" y="200.66" rot="MR90"/>
+<instance part="C4" gate="G$1" x="241.3" y="27.94"/>
+<instance part="GND21" gate="1" x="241.3" y="20.32"/>
 </instances>
 <busses>
@@
 </segment>
 </net>
-<net name="+5V" class="0">
+<net name="+5V" class="1">
 <segment>
 <pinref part="JP6" gate="G$1" pin="3"/>
@@
 </segment>
 <segment>
-<pinref part="X4" gate="G$1" pin="1"/>
-<wire x1="297.18" y1="30.48" x2="281.94" y2="30.48" width="0.1524" layer="91"/>
-<pinref part="P+11" gate="1" pin="+5V"/>
-</segment>
-<segment>
 <pinref part="C3" gate="G$1" pin="+"/>
 <pinref part="P+12" gate="1" pin="+5V"/>
-<wire x1="233.68" y1="38.1" x2="233.68" y2="35.56" width="0.1524" layer="91"/>
+<wire x1="213.36" y1="38.1" x2="213.36" y2="35.56" width="0.1524" layer="91"/>
 </segment>
 </net>
@@
 </segment>
 </net>
-<net name="+3V3" class="0">
+<net name="+3V3" class="1">
 <segment>
 <pinref part="+3V4" gate="G$1" pin="+3V3"/>
@@
 <segment>
 <pinref part="GND10" gate="1" pin="GND"/>
-<wire x1="264.16" y1="27.94" x2="264.16" y2="33.02" width="0.1524" layer="91"/>
+<wire x1="264.16" y1="22.86" x2="264.16" y2="33.02" width="0.1524" layer="91"/>
 <pinref part="X4" gate="G$1" pin="4"/>
 <wire x1="264.16" y1="33.02" x2="266.7" y2="33.02" width="0.1524" layer="91"/>
@@
 <pinref part="X5" gate="G$1" pin="GND"/>
 <pinref part="GND14" gate="1" pin="GND"/>
+</segment>
+<segment>
+<pinref part="C4" gate="G$1" pin="2"/>
+<pinref part="GND21" gate="1" pin="GND"/>
+<wire x1="241.3" y1="25.4" x2="241.3" y2="22.86" width="0.1524" layer="91"/>
 </segment>
 </net>
@@
 <segment>
 <pinref part="C2" gate="G$1" pin="+"/>
-<wire x1="223.52" y1="35.56" x2="223.52" y2="38.1" width="0.1524" layer="91"/>
-<label x="223.52" y="40.64" size="1.778" layer="95"/>
+<wire x1="203.2" y1="35.56" x2="203.2" y2="38.1" width="0.1524" layer="91"/>
+<label x="203.2" y="40.64" size="1.778" layer="95"/>
 </segment>
 <segment>
@@
 </segment>
 </net>
-<net name="IOREF" class="0">
+<net name="IOREF" class="1">
 <segment>
 <pinref part="JP6" gate="G$1" pin="1"/>
@@
 <wire x1="215.9" y1="154.94" x2="220.98" y2="154.94" width="0.1524" layer="91"/>
 <label x="223.52" y="154.94" size="1.778" layer="95"/>
+</segment>
+<segment>
+<pinref part="X4" gate="G$1" pin="1"/>
+<wire x1="297.18" y1="30.48" x2="281.94" y2="30.48" width="0.1524" layer="91"/>
+<label x="299.72" y="30.48" size="1.778" layer="95"/>
 </segment>
 </net>
@@
 </segment>
 </net>
-<net name="N$10" class="0">
+<net name="N$10" class="1">
 <segment>
 <pinref part="U$13" gate="G$1" pin="A2"/>
@@
 <segment>
 <pinref part="X4" gate="G$1" pin="6"/>
-<wire x1="266.7" y1="35.56" x2="264.16" y2="35.56" width="0.1524" layer="91"/>
-<wire x1="264.16" y1="35.56" x2="264.16" y2="58.42" width="0.1524" layer="91"/>
+<wire x1="266.7" y1="35.56" x2="241.3" y2="35.56" width="0.1524" layer="91"/>
+<wire x1="241.3" y1="35.56" x2="241.3" y2="58.42" width="0.1524" layer="91"/>
 <pinref part="R20" gate="G$1" pin="2"/>
-<wire x1="264.16" y1="58.42" x2="284.48" y2="58.42" width="0.1524" layer="91"/>
+<wire x1="241.3" y1="58.42" x2="284.48" y2="58.42" width="0.1524" layer="91"/>
 <wire x1="284.48" y1="58.42" x2="292.1" y2="58.42" width="0.1524" layer="91"/>
 <wire x1="292.1" y1="58.42" x2="292.1" y2="53.34" width="0.1524" layer="91"/>
@@
 <pinref part="R19" gate="G$1" pin="2"/>
 <wire x1="284.48" y1="53.34" x2="284.48" y2="58.42" width="0.1524" layer="91"/>
-</segment>
-</net>
+<junction x="241.3" y="35.56"/>
+<pinref part="C4" gate="G$1" pin="1"/>
+<wire x1="241.3" y1="35.56" x2="241.3" y2="33.02" width="0.1524" layer="91"/>
+</segment>
+</net>

Commit message: Removed SRF, layout changes. Routing and silkscreen tidying.
Parts:
- removed SRF: SRF-LANDING, Ciseco Footprints:SRF-LANDING
- removed X5: SMA, SteveMarple:CONN-SMATHD-SMD-EDGE
- JP1: value ISP VCC -> MAG VCC
Connections:
- removed net ANTENNA: SRF.ANT, X5.SIGNAL
- new net A6: SENS1.VS, U$13.A6
- net !XRF_RESET: no longer SRF.!RESET
- net +3V3: no longer SRF.3V3
- net GND: no longer SRF.GND, X5.GND
- net IOREF: no longer SENS1.VS
- net RX1: no longer SRF.P0_3/TX
- net TX1: no longer SRF.P0_2/RX
- net XRF_HEARTBEAT: no longer SRF.P1_7/MISO
- net XRF_ON: no longer SRF.P1_3
- net XRF_P1_5: no longer SRF.P1_5/SCK
- net XRF_P1_6: no longer SRF.P1_6/MOSI
- net XRF_SLEEP: no longer SRF.P1_4/SS
Changed lines of the file:
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@@
 <part name="R17" library="SteveMarple" deviceset="RESISTOR" device="1206-HAND" value="510k"/>
 <part name="L2" library="SteveMarple" deviceset="INDUCTOR" device="TH-2MM" value="4u7"/>
-<part name="SRF" library="Ciseco Footprints" deviceset="SRF" device="-LANDING" value=""/>
 <part name="XRF" library="SteveMarple" deviceset="XRF" device="B1" value=""/>
 <part name="U$32" library="SteveMarple" deviceset="PAD" device=""/>
@@
 <part name="GND12" library="supply1" deviceset="GND" device=""/>
 <part name="P+12" library="supply1" deviceset="+5V" device=""/>
-<part name="+3V7" library="supply1" deviceset="+3V3" device=""/>
-<part name="GND13" library="supply1" deviceset="GND" device=""/>
-<part name="X5" library="SteveMarple" deviceset="CONN-SMA" device="THD-SMD-EDGE" value="SMA"/>
-<part name="GND14" library="supply1" deviceset="GND" device=""/>
-<part name="JP1" library="SparkFun" deviceset="JUMPER-3" device="PTH" value="ISP VCC"/>
+<part name="JP1" library="SparkFun" deviceset="JUMPER-3" device="PTH" value="MAG VCC"/>
 <part name="C4" library="SparkFun" deviceset="CAP" device="PTH" value="100n"/>
 <part name="GND21" library="supply1" deviceset="GND" device=""/>
@@
 <instance part="R17" gate="G$1" x="119.38" y="30.48" rot="R90"/>
 <instance part="L2" gate="G$1" x="91.44" y="68.58"/>
-<instance part="SRF" gate="G$1" x="261.62" y="-116.84"/>
 <instance part="XRF" gate="G$1" x="264.16" y="-53.34"/>
 <instance part="U$32" gate="G$1" x="238.76" y="-55.88" rot="R180"/>
@@
 <instance part="GND12" gate="1" x="213.36" y="25.4"/>
 <instance part="P+12" gate="1" x="213.36" y="40.64"/>
-<instance part="+3V7" gate="G$1" x="231.14" y="-96.52"/>
-<instance part="GND13" gate="1" x="231.14" y="-129.54"/>
-<instance part="X5" gate="G$1" x="205.74" y="-104.14" rot="MR0"/>
-<instance part="GND14" gate="1" x="205.74" y="-111.76"/>
 <instance part="JP1" gate="G$1" x="309.88" y="200.66" rot="MR90"/>
 <instance part="C4" gate="G$1" x="241.3" y="27.94"/>
@@
 <wire x1="261.62" y1="38.1" x2="261.62" y2="43.18" width="0.1524" layer="91"/>
 </segment>
-<segment>
-<pinref part="SRF" gate="G$1" pin="3V3"/>
-<pinref part="+3V7" gate="G$1" pin="+3V3"/>
-<wire x1="233.68" y1="-106.68" x2="231.14" y2="-106.68" width="0.1524" layer="91"/>
-<wire x1="231.14" y1="-106.68" x2="231.14" y2="-99.06" width="0.1524" layer="91"/>
-</segment>
 </net>
 <net name="GND" class="1">
@@
 <pinref part="C3" gate="G$1" pin="-"/>
 <pinref part="GND12" gate="1" pin="GND"/>
-</segment>
-<segment>
-<pinref part="SRF" gate="G$1" pin="GND"/>
-<pinref part="GND13" gate="1" pin="GND"/>
-<wire x1="233.68" y1="-109.22" x2="231.14" y2="-109.22" width="0.1524" layer="91"/>
-<wire x1="231.14" y1="-109.22" x2="231.14" y2="-127" width="0.1524" layer="91"/>
-</segment>
-<segment>
-<pinref part="X5" gate="G$1" pin="GND"/>
-<pinref part="GND14" gate="1" pin="GND"/>
 </segment>
 <segment>
@@
 <label x="289.56" y="-60.96" size="1.778" layer="95"/>
 </segment>
-<segment>
-<pinref part="SRF" gate="G$1" pin="P1_3"/>
-<wire x1="233.68" y1="-111.76" x2="228.6" y2="-111.76" width="0.1524" layer="91"/>
-<label x="226.06" y="-111.76" size="1.778" layer="95" rot="MR0"/>
-</segment>
 </net>
 <net name="!RESET" class="0">
@@
 <wire x1="243.84" y1="-53.34" x2="231.14" y2="-53.34" width="0.1524" layer="91"/>
 </segment>
-<segment>
-<pinref part="SRF" gate="G$1" pin="!RESET"/>
-<wire x1="254" y1="-127" x2="254" y2="-129.54" width="0.1524" layer="91"/>
-<label x="254" y="-132.08" size="1.778" layer="95" rot="MR0"/>
-</segment>
 </net>
 <net name="XRF_SLEEP" class="0">
@@
 <label x="228.6" y="-63.5" size="1.778" layer="95" rot="MR0"/>
 <pinref part="XRF" gate="G$1" pin="P1_4"/>
-</segment>
-<segment>
-<pinref part="SRF" gate="G$1" pin="P1_4/SS"/>
-<wire x1="233.68" y1="-119.38" x2="228.6" y2="-119.38" width="0.1524" layer="91"/>
-<label x="226.06" y="-119.38" size="1.778" layer="95" rot="MR0"/>
 </segment>
 </net>
@@
 <wire x1="45.72" y1="147.32" x2="55.88" y2="147.32" width="0.1524" layer="91"/>
 <label x="45.72" y="152.4" size="1.778" layer="95" rot="R90"/>
-</segment>
-<segment>
-<wire x1="358.14" y1="157.48" x2="363.22" y2="157.48" width="0.1524" layer="91"/>
-<label x="365.76" y="157.48" size="1.778" layer="95"/>
-<pinref part="SENS1" gate="G$1" pin="VS"/>
 </segment>
 <segment>
@@
 <label x="228.6" y="-58.42" size="1.778" layer="95" rot="MR0"/>
 </segment>
-<segment>
-<pinref part="SRF" gate="G$1" pin="P1_6/MOSI"/>
-<wire x1="233.68" y1="-114.3" x2="228.6" y2="-114.3" width="0.1524" layer="91"/>
-<label x="226.06" y="-114.3" size="1.778" layer="95" rot="MR0"/>
-</segment>
 </net>
 <net name="XRF_P1_5" class="0">
@@
 <label x="228.6" y="-60.96" size="1.778" layer="95" rot="MR0"/>
 </segment>
-<segment>
-<pinref part="SRF" gate="G$1" pin="P1_5/SCK"/>
-<wire x1="233.68" y1="-116.84" x2="228.6" y2="-116.84" width="0.1524" layer="91"/>
-<label x="226.06" y="-116.84" size="1.778" layer="95" rot="MR0"/>
-</segment>
 </net>
 <net name="N$25" class="0">
@@
 <label x="228.6" y="-45.72" size="1.778" layer="95" rot="MR0"/>
 </segment>
-<segment>
-<pinref part="SRF" gate="G$1" pin="P0_3/TX"/>
-<wire x1="289.56" y1="-114.3" x2="292.1" y2="-114.3" width="0.1524" layer="91"/>
-<label x="294.64" y="-114.3" size="1.778" layer="95"/>
-</segment>
 </net>
 <net name="TX1" class="0">
@@
 <wire x1="243.84" y1="-48.26" x2="231.14" y2="-48.26" width="0.1524" layer="91"/>
 <label x="228.6" y="-48.26" size="1.778" layer="95" rot="MR0"/>
-</segment>
-<segment>
-<pinref part="SRF" gate="G$1" pin="P0_2/RX"/>
-<wire x1="289.56" y1="-116.84" x2="292.1" y2="-116.84" width="0.1524" layer="91"/>
-<label x="294.64" y="-116.84" size="1.778" layer="95"/>
 </segment>
 </net>
@@
 </segment>
 </net>
-<net name="ANTENNA" class="2">
-<segment>
-<pinref part="SRF" gate="G$1" pin="ANT"/>
-<pinref part="X5" gate="G$1" pin="SIGNAL"/>
-<wire x1="210.82" y1="-104.14" x2="233.68" y2="-104.14" width="0.1524" layer="91"/>
-</segment>
-</net>
 <net name="XRF_HEARTBEAT" class="0">
-<segment>
-<pinref part="SRF" gate="G$1" pin="P1_7/MISO"/>
-<wire x1="289.56" y1="-119.38" x2="292.1" y2="-119.38" width="0.1524" layer="91"/>
-<label x="294.64" y="-119.38" size="1.778" layer="95"/>
-</segment>
 <segment>
 <pinref part="XRF" gate="G$1" pin="HEARTBEAT"/>
@@
 </segment>
 </net>
-<net name="N$7" class="0">
+<net name="N$7" class="1">
 <segment>
 <pinref part="X1" gate="G$1" pin="8"/>
@@
 </segment>
 </net>
+<net name="A6" class="0">
+<segment>
+<wire x1="358.14" y1="157.48" x2="363.22" y2="157.48" width="0.1524" layer="91"/>
+<label x="365.76" y="157.48" size="1.778" layer="95"/>
+<pinref part="SENS1" gate="G$1" pin="VS"/>
+</segment>
+<segment>
+<pinref part="U$13" gate="G$1" pin="A6"/>
+<wire x1="170.18" y1="200.66" x2="160.02" y2="200.66" width="0.1524" layer="91"/>
+<label x="157.48" y="200.66" size="1.778" layer="95" rot="MR0"/>
+</segment>
+</net>

Commit message: Minor adjustments for PCB layout.
Parts:
- removed U$15: PAD, SteveMarple:PAD
- added U$2, U$4: PAD, SteveMarple:PAD
- C3: value 4u7 25V -> 4u7
- IC4: value MCP1640SOT23-6-HAND -> MCP1640
Connections:
- net GND: no longer U$15.1
- net XRF_P1_5: now also U$4.1
- net XRF_P1_6: now also U$2.1
Changed lines of the file:
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@@
 <part name="U$6" library="SteveMarple" deviceset="PAD" device=""/>
 <part name="GND15" library="supply1" deviceset="GND" device=""/>
-<part name="U$15" library="SteveMarple" deviceset="PAD" device=""/>
 <part name="U$16" library="SteveMarple" deviceset="PAD" device=""/>
 <part name="+3V4" library="supply1" deviceset="+3V3" device=""/>
@@
 <part name="JP9" library="SparkFun" deviceset="JUMPER-2" device="PTH" value="CLOUD PWR"/>
 <part name="JP11" library="pinhead" deviceset="PINHD-2X3" device="" value="ALT ISP"/>
-<part name="IC4" library="SteveMarple" deviceset="MCP1640" device="SOT23-6-HAND" value="MCP1640SOT23-6-HAND"/>
+<part name="IC4" library="SteveMarple" deviceset="MCP1640" device="SOT23-6-HAND" value="MCP1640"/>
 <part name="GND17" library="supply1" deviceset="GND" device=""/>
 <part name="C15" library="SteveMarple" deviceset="C-EU" device="1206-HAND" value="4u7"/>
@@
 <part name="R20" library="SteveMarple" deviceset="RESISTOR" device="" value="10k"/>
 <part name="P+6" library="supply1" deviceset="+5V" device=""/>
-<part name="C3" library="SparkFun" deviceset="CAP_POL" device="PTH2" value="4u7 25V"/>
+<part name="C3" library="SparkFun" deviceset="CAP_POL" device="PTH2" value="4u7"/>
 <part name="GND12" library="supply1" deviceset="GND" device=""/>
 <part name="P+12" library="supply1" deviceset="+5V" device=""/>
@@
 <part name="C4" library="SparkFun" deviceset="CAP" device="PTH" value="100n"/>
 <part name="GND21" library="supply1" deviceset="GND" device=""/>
+<part name="U$2" library="SteveMarple" deviceset="PAD" device=""/>
+<part name="U$4" library="SteveMarple" deviceset="PAD" device=""/>
 </parts>
 <sheets>
@@
 <instance part="U$6" gate="G$1" x="165.1" y="226.06"/>
 <instance part="GND15" gate="1" x="208.28" y="137.16"/>
-<instance part="U$15" gate="G$1" x="210.82" y="142.24"/>
 <instance part="U$16" gate="G$1" x="213.36" y="142.24"/>
 <instance part="+3V4" gate="G$1" x="144.78" y="243.84"/>
@@
 <instance part="C4" gate="G$1" x="241.3" y="27.94"/>
 <instance part="GND21" gate="1" x="241.3" y="20.32"/>
+<instance part="U$2" gate="G$1" x="238.76" y="-58.42" rot="R180"/>
+<instance part="U$4" gate="G$1" x="238.76" y="-60.96" rot="R180"/>
 </instances>
 <busses>
@@
 <pinref part="GND15" gate="1" pin="GND"/>
 <wire x1="208.28" y1="139.7" x2="208.28" y2="142.24" width="0.1524" layer="91"/>
-<wire x1="208.28" y1="142.24" x2="210.82" y2="142.24" width="0.1524" layer="91"/>
-<pinref part="U$15" gate="G$1" pin="1"/>
-<wire x1="210.82" y1="142.24" x2="213.36" y2="142.24" width="0.1524" layer="91"/>
-<junction x="210.82" y="142.24"/>
+<wire x1="208.28" y1="142.24" x2="213.36" y2="142.24" width="0.1524" layer="91"/>
 <pinref part="U$16" gate="G$1" pin="1"/>
 </segment>
@@
 <segment>
 <pinref part="XRF" gate="G$1" pin="P1_6"/>
-<wire x1="243.84" y1="-58.42" x2="231.14" y2="-58.42" width="0.1524" layer="91"/>
-<label x="228.6" y="-58.42" size="1.778" layer="95" rot="MR0"/>
+<wire x1="243.84" y1="-58.42" x2="238.76" y2="-58.42" width="0.1524" layer="91"/>
+<pinref part="U$2" gate="G$1" pin="1"/>
 </segment>
 </net>
@@
 <segment>
 <pinref part="XRF" gate="G$1" pin="P1_5"/>
-<wire x1="243.84" y1="-60.96" x2="231.14" y2="-60.96" width="0.1524" layer="91"/>
-<label x="228.6" y="-60.96" size="1.778" layer="95" rot="MR0"/>
-</segment>
-</net>
+<wire x1="243.84" y1="-60.96" x2="238.76" y2="-60.96" width="0.1524" layer="91"/>
+<pinref part="U$4" gate="G$1" pin="1"/>
+</segment>
+</net>

Commit message: Minor routing changes.
Parts:
- JP9: value CLOUD PWR -> CLOUD CTRL
Changed lines of the file:
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@@
 <part name="+3V3" library="supply1" deviceset="+3V3" device=""/>
 <part name="GND4" library="supply1" deviceset="GND" device=""/>
-<part name="JP9" library="SparkFun" deviceset="JUMPER-2" device="PTH" value="CLOUD PWR"/>
+<part name="JP9" library="SparkFun" deviceset="JUMPER-2" device="PTH" value="CLOUD CTRL"/>
 <part name="JP11" library="pinhead" deviceset="PINHD-2X3" device="" value="ALT ISP"/>
 <part name="IC4" library="SteveMarple" deviceset="MCP1640" device="SOT23-6-HAND" value="MCP1640"/>
