File: hardware/FLC100_shield/shield_v2.0/FLC100_shield_v2.0.sch (EAGLE design)
At the start: 68 parts, among them IC1 TSR 1-2450, IC4 MCP1640, J1 RJ11-6PTH, Q1 2N7000, Q2 2N7000, Q3 2N7000, Q4 2N7000, Q5 2N7000, Q6 2N7000, Q7 2N7000, Q8 2N7000, Q9 2N7000, X1 RJ45, X2 CLOUD SENSOR, X4 HUMIDITY

Commit message: Providing options for cloud detector level shifting pull-up voltage.
Parts:
- added D1, D2: BAT85, SteveMarple:DIODE-SCHOTTKY
Connections:
- new net CLOUD_PULLUP: D1.C, D2.C, R10.2, R13.2
- net +5V: now also X3.1, X3.2; no longer R10.2, R13.2, R2.2, R6.2
- net CLOUD_VCC: now also D2.A
- net IOREF: now also D1.A
- net MAG_VCC: now also R2.2, R6.2
Other:
- note added: "Diodes force pull-up to the higher voltage. May omit one diode and replace other by wire link when voltages known in advance."
- moved on the sheet: R10, R13
Changed lines of the file:
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@@
 <setting verticaltext="up"/>
 </settings>
-<grid distance="0.1" unitdist="inch" unit="inch" style="lines" multiple="1" display="no" altdistance="0.01" altunitdist="inch" altunit="inch"/>
+<grid distance="0.1" unitdist="inch" unit="inch" style="lines" multiple="1" display="yes" altdistance="0.01" altunitdist="inch" altunit="inch"/>
 <layers>
 <layer number="1" name="Top" color="4" fill="1" visible="no" active="no"/>
@@
 <part name="GND1" library="supply1" deviceset="GND" device=""/>
 <part name="GND2" library="supply1" deviceset="GND" device=""/>
-<part name="P+3" library="supply1" deviceset="+5V" device=""/>
-<part name="P+4" library="supply1" deviceset="+5V" device=""/>
 <part name="J1" library="SparkFun" deviceset="RJ11-6" device="PTH"/>
 <part name="MOD-1016" library="SteveMarple" deviceset="EMBEDDED_ADVENTURES_MOD-1016" device="NO-HOLES" value=""/>
@@
 <part name="R11" library="SteveMarple" deviceset="RESISTOR" device="" value="10k"/>
 <part name="R14" library="SteveMarple" deviceset="RESISTOR" device="" value="10k"/>
-<part name="P+8" library="supply1" deviceset="+5V" device=""/>
-<part name="P+9" library="supply1" deviceset="+5V" device=""/>
 <part name="R4" library="SteveMarple" deviceset="RESISTOR" device="" value="1k"/>
 <part name="X2" library="SteveMarple" deviceset="ML8" device="" value="CLOUD SENSOR"/>
@@
 <part name="U$2" library="SteveMarple" deviceset="PAD" device=""/>
 <part name="U$4" library="SteveMarple" deviceset="PAD" device=""/>
+<part name="D1" library="SteveMarple" deviceset="DIODE-SCHOTTKY" device="" value="BAT85"/>
+<part name="D2" library="SteveMarple" deviceset="DIODE-SCHOTTKY" device="" value="BAT85"/>
+<part name="P+3" library="supply1" deviceset="+5V" device=""/>
+<part name="P+4" library="supply1" deviceset="+5V" device=""/>
 </parts>
 <sheets>
@@
 <text x="317.5" y="30.48" size="1.778" layer="91">No level-shifting so maximum pull-up
 voltage should be IOREF.</text>
+<text x="76.2" y="160.02" size="1.27" layer="91" align="top-left">Diodes force pull-up to the higher voltage.
+May omit one diode and replace other by
+wire link when voltages known in advance.</text>
 </plain>
 <instances>
@@
 <instance part="GND1" gate="1" x="175.26" y="73.66"/>
 <instance part="GND2" gate="1" x="198.12" y="73.66"/>
-<instance part="P+3" gate="1" x="71.12" y="243.84"/>
-<instance part="P+4" gate="1" x="71.12" y="205.74"/>
 <instance part="J1" gate="G$1" x="304.8" y="182.88" rot="R180"/>
 <instance part="MOD-1016" gate="G$1" x="287.02" y="78.74"/>
@@
 <instance part="Q8" gate="G$1" x="58.42" y="93.98" rot="R270"/>
 <instance part="Q9" gate="G$1" x="83.82" y="93.98" rot="MR270"/>
-<instance part="R10" gate="G$1" x="71.12" y="139.7" rot="R90"/>
-<instance part="R13" gate="G$1" x="71.12" y="101.6" rot="R90"/>
+<instance part="R10" gate="G$1" x="68.58" y="139.7" rot="R90"/>
+<instance part="R13" gate="G$1" x="73.66" y="101.6" rot="R90"/>
 <instance part="R9" gate="G$1" x="45.72" y="139.7" rot="R90"/>
 <instance part="R12" gate="G$1" x="45.72" y="101.6" rot="R90"/>
 <instance part="R11" gate="G$1" x="96.52" y="139.7" rot="R90"/>
 <instance part="R14" gate="G$1" x="96.52" y="101.6" rot="R90"/>
-<instance part="P+8" gate="1" x="71.12" y="149.86"/>
-<instance part="P+9" gate="1" x="71.12" y="111.76"/>
 <instance part="R4" gate="G$1" x="284.48" y="228.6" rot="MR0"/>
 <instance part="X2" gate="G$1" x="271.78" y="124.46"/>
@@
 <instance part="U$2" gate="G$1" x="238.76" y="-58.42" rot="R180"/>
 <instance part="U$4" gate="G$1" x="238.76" y="-60.96" rot="R180"/>
+<instance part="D1" gate="G$1" x="60.96" y="147.32"/>
+<instance part="D2" gate="G$1" x="81.28" y="147.32" rot="MR0"/>
+<instance part="P+3" gate="1" x="175.26" y="129.54"/>
+<instance part="P+4" gate="1" x="198.12" y="129.54"/>
 </instances>
 <busses>
@@
 </segment>
 <segment>
-<pinref part="R2" gate="G$1" pin="2"/>
-<wire x1="71.12" y1="241.3" x2="71.12" y2="238.76" width="0.1524" layer="91"/>
-<pinref part="P+3" gate="1" pin="+5V"/>
-</segment>
-<segment>
-<pinref part="R6" gate="G$1" pin="2"/>
-<wire x1="71.12" y1="203.2" x2="71.12" y2="200.66" width="0.1524" layer="91"/>
-<pinref part="P+4" gate="1" pin="+5V"/>
-</segment>
-<segment>
 <pinref part="IC1" gate="G$1" pin="OUT"/>
 <wire x1="368.3" y1="99.06" x2="368.3" y2="91.44" width="0.1524" layer="91"/>
 <wire x1="368.3" y1="91.44" x2="365.76" y2="91.44" width="0.1524" layer="91"/>
 <pinref part="P+7" gate="1" pin="+5V"/>
-</segment>
-<segment>
-<pinref part="R10" gate="G$1" pin="2"/>
-<wire x1="71.12" y1="147.32" x2="71.12" y2="144.78" width="0.1524" layer="91"/>
-<pinref part="P+8" gate="1" pin="+5V"/>
-</segment>
-<segment>
-<pinref part="R13" gate="G$1" pin="2"/>
-<wire x1="71.12" y1="109.22" x2="71.12" y2="106.68" width="0.1524" layer="91"/>
-<pinref part="P+9" gate="1" pin="+5V"/>
 </segment>
 <segment>
@@
 <pinref part="P+12" gate="1" pin="+5V"/>
 <wire x1="213.36" y1="38.1" x2="213.36" y2="35.56" width="0.1524" layer="91"/>
+</segment>
+<segment>
+<pinref part="P+3" gate="1" pin="+5V"/>
+<wire x1="175.26" y1="127" x2="175.26" y2="121.92" width="0.1524" layer="91"/>
+<pinref part="X3" gate="A" pin="1"/>
+<wire x1="175.26" y1="121.92" x2="182.88" y2="121.92" width="0.1524" layer="91"/>
+</segment>
+<segment>
+<pinref part="X3" gate="A" pin="2"/>
+<wire x1="190.5" y1="121.92" x2="198.12" y2="121.92" width="0.1524" layer="91"/>
+<pinref part="P+4" gate="1" pin="+5V"/>
+<wire x1="198.12" y1="121.92" x2="198.12" y2="127" width="0.1524" layer="91"/>
 </segment>
 </net>
@@
 </segment>
 </net>
-<net name="ISP_VCC" class="0">
+<net name="ISP_VCC" class="1">
 <segment>
 <pinref part="U$13" gate="G$1" pin="ISP_VCC"/>
@@
 <wire x1="45.72" y1="147.32" x2="55.88" y2="147.32" width="0.1524" layer="91"/>
 <label x="45.72" y="152.4" size="1.778" layer="95" rot="R90"/>
+<junction x="55.88" y="147.32"/>
+<pinref part="D1" gate="G$1" pin="A"/>
 </segment>
 <segment>
@@
 <wire x1="86.36" y1="241.3" x2="96.52" y2="241.3" width="0.1524" layer="91"/>
 <label x="109.22" y="241.3" size="1.778" layer="95"/>
+<junction x="86.36" y="241.3"/>
+<pinref part="R2" gate="G$1" pin="2"/>
+<wire x1="71.12" y1="238.76" x2="71.12" y2="241.3" width="0.1524" layer="91"/>
+<wire x1="71.12" y1="241.3" x2="86.36" y2="241.3" width="0.1524" layer="91"/>
 </segment>
 <segment>
@@
 <wire x1="86.36" y1="203.2" x2="96.52" y2="203.2" width="0.1524" layer="91"/>
 <label x="109.22" y="203.2" size="1.778" layer="95"/>
+<junction x="86.36" y="203.2"/>
+<pinref part="R6" gate="G$1" pin="2"/>
+<wire x1="71.12" y1="200.66" x2="71.12" y2="203.2" width="0.1524" layer="91"/>
+<wire x1="71.12" y1="203.2" x2="86.36" y2="203.2" width="0.1524" layer="91"/>
 </segment>
 <segment>
@@
 <pinref part="Q6" gate="G$1" pin="D"/>
 <pinref part="Q7" gate="G$1" pin="D"/>
-<wire x1="63.5" y1="132.08" x2="71.12" y2="132.08" width="0.1524" layer="91"/>
-<junction x="71.12" y="132.08"/>
-<wire x1="71.12" y1="132.08" x2="78.74" y2="132.08" width="0.1524" layer="91"/>
+<wire x1="63.5" y1="132.08" x2="68.58" y2="132.08" width="0.1524" layer="91"/>
+<junction x="68.58" y="132.08"/>
+<wire x1="68.58" y1="132.08" x2="78.74" y2="132.08" width="0.1524" layer="91"/>
 <pinref part="R10" gate="G$1" pin="1"/>
-<wire x1="71.12" y1="132.08" x2="71.12" y2="134.62" width="0.1524" layer="91"/>
+<wire x1="68.58" y1="132.08" x2="68.58" y2="134.62" width="0.1524" layer="91"/>
 </segment>
 </net>
@@
 <pinref part="Q8" gate="G$1" pin="D"/>
 <pinref part="Q9" gate="G$1" pin="D"/>
-<wire x1="63.5" y1="93.98" x2="71.12" y2="93.98" width="0.1524" layer="91"/>
+<wire x1="63.5" y1="93.98" x2="73.66" y2="93.98" width="0.1524" layer="91"/>
 <pinref part="R13" gate="G$1" pin="1"/>
-<wire x1="71.12" y1="93.98" x2="78.74" y2="93.98" width="0.1524" layer="91"/>
-<wire x1="71.12" y1="93.98" x2="71.12" y2="96.52" width="0.1524" layer="91"/>
-<junction x="71.12" y="93.98"/>
+<wire x1="73.66" y1="93.98" x2="78.74" y2="93.98" width="0.1524" layer="91"/>
+<wire x1="73.66" y1="93.98" x2="73.66" y2="96.52" width="0.1524" layer="91"/>
+<junction x="73.66" y="93.98"/>
 </segment>
 </net>
@@
 <wire x1="86.36" y1="147.32" x2="96.52" y2="147.32" width="0.1524" layer="91"/>
 <label x="109.22" y="147.32" size="1.778" layer="95"/>
+<junction x="86.36" y="147.32"/>
+<pinref part="D2" gate="G$1" pin="A"/>
 </segment>
 <segment>
@@
 </segment>
 </net>
+<net name="CLOUD_PULLUP" class="0">
+<segment>
+<pinref part="R10" gate="G$1" pin="2"/>
+<wire x1="68.58" y1="147.32" x2="68.58" y2="144.78" width="0.1524" layer="91"/>
+<pinref part="R13" gate="G$1" pin="2"/>
+<wire x1="73.66" y1="147.32" x2="73.66" y2="106.68" width="0.1524" layer="91"/>
+<wire x1="68.58" y1="147.32" x2="71.12" y2="147.32" width="0.1524" layer="91"/>
+<junction x="71.12" y="147.32"/>
+<wire x1="71.12" y1="147.32" x2="73.66" y2="147.32" width="0.1524" layer="91"/>
+<wire x1="71.12" y1="147.32" x2="71.12" y2="149.86" width="0.1524" layer="91"/>
+<label x="71.12" y="149.86" size="1.778" layer="95" rot="R90"/>
+<junction x="68.58" y="147.32"/>
+<junction x="73.66" y="147.32"/>
+<pinref part="D1" gate="G$1" pin="C"/>
+<wire x1="68.58" y1="147.32" x2="66.04" y2="147.32" width="0.1524" layer="91"/>
+<pinref part="D2" gate="G$1" pin="C"/>
+<wire x1="73.66" y1="147.32" x2="76.2" y2="147.32" width="0.1524" layer="91"/>
+</segment>
+</net>

Commit message: Change footprint for Vin capacitor to ensure 25V rating can be achieved.
Parts:
- removed C15: 4u7, SteveMarple:C-EU1206-HAND
- removed C9: 100n, SparkFun:CAPPTH
- removed IC4: MCP1640, SteveMarple:MCP1640SOT23-6-HAND
- removed J1: RJ11-6PTH, SparkFun:RJ11-6PTH
- removed JP13: VIN ADC, SparkFun:JUMPER-2PTH
- removed JP9: CLOUD CTRL, SparkFun:JUMPER-2PTH
- removed MOD-1016: EMBEDDED_ADVENTURES_MOD-1016NO-HOLES, SteveMarple:EMBEDDED_ADVENTURES_MOD-1016NO-HOLES
- removed R20: 10k, SteveMarple:RESISTOR
- removed U$16, U$22, U$23, U$25, U$32, U$40: PAD, SteveMarple:PAD
- added C6: 4u7 25V, SteveMarple:CAP_POL
- added C7: 4u7, SteveMarple:CAP_POLPTH2
- added IC2: TSR 1-2450, SteveMarple:V_REG_78XXSIDE
- added JP3: MAG VCC, SparkFun:JUMPER-3PTH
- added JP5: ISP VCC, SparkFun:JUMPER-3PTH
- added MOD-1: EMBEDDED_ADVENTURES_MOD-1016NO-HOLES, SteveMarple:EMBEDDED_ADVENTURES_MOD-1016NO-HOLES
- added R18: 15k, SteveMarple:RESISTOR1206-HAND
- added U$10, U$11, U$12, U$7, U$8, U$9: PAD, SteveMarple:PAD
- added X5: HUMIDITY, SteveMarple:ML8
- C2: value 4u7 25V -> 100u; device SparkFun:CAP_POLPTH2 -> SteveMarple:CAP_POLPTH2
- C3: value 4u7 -> 100n; device SparkFun:CAP_POLPTH2 -> SparkFun:CAPPTH
- C4: value 100n -> 4u7; device SparkFun:CAPPTH -> SteveMarple:C-EU1206-HAND
- C8: value 100u -> 100n; device SparkFun:CAP_POLPTH2 -> SparkFun:CAPPTH
- IC1: value TSR 1-2450 -> MCP1640; device SteveMarple:V_REG_78XXSIDE -> SteveMarple:MCP1640SOT23-6-HAND
- JP1: value MAG VCC -> 5V LINK; device SparkFun:JUMPER-3PTH -> SparkFun:JUMPER-2PTH
- JP2: value 5V LINK -> VIN ADC
- JP6: value ISP VCC -> CLOUD CTRL; device SparkFun:JUMPER-3PTH -> SparkFun:JUMPER-2PTH
- R15: value 910k -> 10k; device SteveMarple:RESISTOR1206-HAND -> SteveMarple:RESISTOR
- R16: value 15k -> 10k; device SteveMarple:RESISTOR1206-HAND -> SteveMarple:RESISTOR
- R17: value 510k -> 910k
- R19: value 10k -> 510k; device SteveMarple:RESISTOR -> SteveMarple:RESISTOR1206-HAND
- U$13: value CALUNIUM-SHIELD-V3 -> PAD; device SteveMarple:CALUNIUM-SHIELD-V3V3-NO-HOLES-NO-TEXT -> SteveMarple:PAD
- U$4: value PAD -> CALUNIUM-SHIELD-V3; device SteveMarple:PAD -> SteveMarple:CALUNIUM-SHIELD-V3V3-NO-HOLES-NO-TEXT
- X2: value CLOUD SENSOR -> RJ11; device SteveMarple:ML8 -> SteveMarple:RJ11-6PTH
- X3: value (none) -> CLOUD SENSOR; device pinhead:PINHD-2X18 -> SteveMarple:ML8
- X4: value HUMIDITY -> MEGA2560; device SteveMarple:ML8 -> pinhead:PINHD-2X18
- renumbered C16 to C5, JP11 to JP4, L2 to L1
Connections:
- net !RESET: now also U$4.!RESET@0, U$4.!RESET@1; no longer U$13.!RESET@0, U$13.!RESET@1
- net !XRF_RESET: now also U$4.5; no longer U$13.5
- net +3V3: now also C2.+, C3.1, IC1.VOUT, JP3.3, R17.2, U$3.1, U$4.3.3V, X3.8, X5.8; no longer C8.+, C9.1, IC4.VOUT, JP1.3, R15.2, U$13.3.3V, U$22.1, X2.8, X4.8
- net +5V: now also C7.+, IC2.OUT, JP1.1, JP5.3, U$2.1, U$4.5V, X4.1, X4.2; no longer C3.+, IC1.OUT, JP2.1, JP6.3, U$13.5V, U$3.1, X2.1, X3.2
- net 11: now also U$4.11(MOSI); no longer U$13.11(MOSI)
- net 12: now also U$4.12(MISO); no longer U$13.12(MISO)
- net 13: now also U$4.13(SCK); no longer U$13.13(SCK)
- net 14: now also MOD-1.SDA_MOSI, U$4.14; no longer MOD-1016.SDA_MOSI, U$13.14
- net 16: now also U$4.16; no longer U$13.16
- net 17: now also MOD-1.SCL, U$4.17; no longer MOD-1016.SCL, U$13.17
- net 18: now also JP6.1, U$4.18; no longer JP9.1, U$13.18
- net 19: now also U$4.19; no longer U$13.19
- net 6: now also MOD-1.IRQ, U$4.6; no longer MOD-1016.IRQ, U$13.6
- net A6: now also U$4.A6; no longer U$13.A6
- net A7: now also U$4.A7; no longer U$13.A7
- net CLOUD_SCL: now also X3.5; no longer X2.5
- net CLOUD_SDA: now also X3.7; no longer X2.7
- net CLOUD_VCC: now also X3.6; no longer X2.6
- net GND: now also C3.2, C6.-, C7.-, C8.2, IC2.GND, MOD-1.GND, R19.1, U$12.1, U$14.1, U$4.GND, X2.3, X3.4, X4.35, X4.36, X5.4; no longer C15.2, C3.-, C8.-, C9.2, IC4.GND, J1.3, MOD-1016.GND, R17.1, U$13.GND, U$16.1, U$40.1, X2.4, X3.35, X3.36, X4.4
- net HUMIDITY_SCL: now also R16.1, U$4.A5, X5.5; no longer R20.1, U$13.A5, X4.5
- net HUMIDITY_SDA: now also R15.1, U$4.A4, X5.7; no longer R19.1, U$13.A4, X4.7
- net IOREF: now also JP5.1, MOD-1.VCC, U$4.IOREF, U$5.1, X5.1; no longer JP6.1, MOD-1016.VCC, U$13.IOREF, U$14.1, X4.1
- net ISP_VCC: now also JP5.2, U$4.ISP_VCC; no longer JP6.2, U$13.ISP_VCC
- net MAG_SCL: now also X2.4; no longer J1.4
- net MAG_SDA: now also X2.6; no longer J1.6
- net MAG_VCC: now also JP1.2, X2.5; no longer J1.5, JP2.2
- net MISO: now also U$4.ISP_MISO, X4.31; no longer U$13.ISP_MISO, X3.31
- net MOSI: now also U$4.ISP_MOSI, X4.32; no longer U$13.ISP_MOSI, X3.32
- net N$10: now also JP2.2, U$4.A2; no longer JP13.2, U$13.A2
- net N$16: now also U$13.1, X5.3; no longer U$5.1, X4.3
- net N$22: now also C8.1, R15.2, R16.2, X5.6; no longer C4.1, R19.2, R20.2, X4.6
- net N$25: now also U$8.1; no longer U$25.1
- net N$26: now also U$4.9; no longer U$13.9
- net N$27: now also U$7.1; no longer U$23.1
- net N$3: now also JP6.2, X3.3; no longer JP9.2, X2.3
- net N$41: now also IC1.SW; no longer IC4.SW
- net N$42: now also R18.1, R19.2; no longer R16.1, R17.2
- net N$46: now also IC1.VFB, R17.1, R18.2; no longer IC4.VFB, R15.1, R16.2
- net N$6: now also X2.2; no longer J1.2
- net N$7: now also JP3.2; no longer JP1.2
- net RX1: now also U$4.2(RX1)@1; no longer U$13.2(RX1)@1
- net SCK: now also U$4.ISP_SCK, X4.33; no longer U$13.ISP_SCK, X3.33
- net SCL: now also U$4.21(SCL)@1; no longer U$13.21(SCL)@1
- net SDA: now also U$4.20(SDA)@1; no longer U$13.20(SDA)@1
- net TX1: now also U$4.3(TX1)@1; no longer U$13.3(TX1)@1
- net VIN: now also C4.1, C6.+, IC1.EN, IC1.VIN, IC2.IN, JP2.1, JP3.1, U$4.VIN, X2.1, X3.2, X5.2; no longer C15.1, C2.+, IC1.IN, IC4.EN, IC4.VIN, J1.1, JP1.1, JP13.1, U$13.VIN, X2.2, X4.2
- net XRF_HEARTBEAT: now also U$9.1; no longer U$32.1
- net XRF_ON: now also U$4.23; no longer U$13.23
- net XRF_P1_5: now also U$11.1; no longer U$4.1
- net XRF_P1_6: now also U$10.1; no longer U$2.1
- net XRF_SLEEP: now also U$4.7; no longer U$13.7
Other:
- note added: "No level-shifting so maximum pull-up voltage should be IOREF. Leave remote board to set operating and pull-up voltages."
- note removed: "Add HIH6136 I2C version (see blog) humidity sensor. Have pull-up resistors at both ends of bus, but pull-up voltage selected on remote PCB. OR - fit HIH6136 sensor on same external PCB as used for the cloud detector?"
- note removed: "Add MLX... IR temp sensor with level shifting and jumper for operating voltage"
- note removed: "Add pinout for 3V3 boost breakout board"
- note removed: "Connect ISP pins"
- note removed: "I2C pull-ups on v1.1 should be to IOREF"
- note removed: "LABEL X2 NETS CORRECTLY"
- note removed: "No level-shifting so maximum pull-up voltage should be IOREF."
- moved on the sheet: C1, C2, C4, JP2, R15, R16, R17, R19, SENS1, XRF
