File: hardware/FLC100_shield/remote_v2/FLC100_remote_v2.sch (EAGLE design)
At the start: 33 parts, among them IC1 MCP3424, IC2 MAX619, IC3 MCP1702-5.0, Q1 2N7000, X1 RJ45

Commit message: Separating supply inputs for linear and boost regulators.
Parts:
- added C10: 4u7, SparkFun:CAP_POLPTH2
Connections:
- new net VIN_ALT: C10.+, IC3.VIN, X1.2
- net GND: now also C10.-
- net VIN: no longer IC3.VIN
Other:
- note removed: "Remote board can be used without ADC and feed analogue signal to FLC100 shield."
Changed lines of the file:
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@@
 <grid distance="0.1" unitdist="inch" unit="inch" style="lines" multiple="1" display="no" altdistance="0.01" altunitdist="inch" altunit="inch"/>
 <layers>
-<layer number="1" name="Top" color="4" fill="1" visible="yes" active="no"/>
-<layer number="2" name="Route2" color="1" fill="3" visible="yes" active="no"/>
-<layer number="3" name="Route3" color="4" fill="3" visible="yes" active="no"/>
-<layer number="14" name="Route14" color="1" fill="6" visible="yes" active="no"/>
-<layer number="15" name="Route15" color="4" fill="6" visible="yes" active="no"/>
-<layer number="16" name="Bottom" color="1" fill="1" visible="yes" active="no"/>
-<layer number="17" name="Pads" color="2" fill="1" visible="yes" active="no"/>
-<layer number="18" name="Vias" color="2" fill="1" visible="yes" active="no"/>
-<layer number="19" name="Unrouted" color="6" fill="1" visible="yes" active="no"/>
-<layer number="20" name="Dimension" color="15" fill="1" visible="yes" active="no"/>
-<layer number="21" name="tPlace" color="7" fill="1" visible="yes" active="no"/>
-<layer number="22" name="bPlace" color="7" fill="1" visible="yes" active="no"/>
-<layer number="23" name="tOrigins" color="15" fill="1" visible="yes" active="no"/>
-<layer number="24" name="bOrigins" color="15" fill="1" visible="yes" active="no"/>
-<layer number="25" name="tNames" color="7" fill="1" visible="yes" active="no"/>
-<layer number="26" name="bNames" color="7" fill="1" visible="yes" active="no"/>
-<layer number="27" name="tValues" color="7" fill="1" visible="yes" active="no"/>
-<layer number="28" name="bValues" color="7" fill="1" visible="yes" active="no"/>
+<layer number="1" name="Top" color="4" fill="1" visible="no" active="no"/>
+<layer number="2" name="Route2" color="1" fill="3" visible="no" active="no"/>
+<layer number="3" name="Route3" color="4" fill="3" visible="no" active="no"/>
+<layer number="14" name="Route14" color="1" fill="6" visible="no" active="no"/>
+<layer number="15" name="Route15" color="4" fill="6" visible="no" active="no"/>
+<layer number="16" name="Bottom" color="1" fill="1" visible="no" active="no"/>
+<layer number="17" name="Pads" color="2" fill="1" visible="no" active="no"/>
+<layer number="18" name="Vias" color="2" fill="1" visible="no" active="no"/>
+<layer number="19" name="Unrouted" color="6" fill="1" visible="no" active="no"/>
+<layer number="20" name="Dimension" color="15" fill="1" visible="no" active="no"/>
+<layer number="21" name="tPlace" color="7" fill="1" visible="no" active="no"/>
+<layer number="22" name="bPlace" color="7" fill="1" visible="no" active="no"/>
+<layer number="23" name="tOrigins" color="15" fill="1" visible="no" active="no"/>
+<layer number="24" name="bOrigins" color="15" fill="1" visible="no" active="no"/>
+<layer number="25" name="tNames" color="7" fill="1" visible="no" active="no"/>
+<layer number="26" name="bNames" color="7" fill="1" visible="no" active="no"/>
+<layer number="27" name="tValues" color="7" fill="1" visible="no" active="no"/>
+<layer number="28" name="bValues" color="7" fill="1" visible="no" active="no"/>
 <layer number="29" name="tStop" color="7" fill="3" visible="no" active="no"/>
 <layer number="30" name="bStop" color="7" fill="6" visible="no" active="no"/>
@@
 <layer number="35" name="tGlue" color="7" fill="4" visible="no" active="no"/>
 <layer number="36" name="bGlue" color="7" fill="5" visible="no" active="no"/>
-<layer number="37" name="tTest" color="7" fill="1" visible="yes" active="no"/>
-<layer number="38" name="bTest" color="7" fill="1" visible="yes" active="no"/>
+<layer number="37" name="tTest" color="7" fill="1" visible="no" active="no"/>
+<layer number="38" name="bTest" color="7" fill="1" visible="no" active="no"/>
 <layer number="39" name="tKeepout" color="4" fill="11" visible="no" active="no"/>
 <layer number="40" name="bKeepout" color="1" fill="11" visible="no" active="no"/>
@@
 <layer number="44" name="Drills" color="7" fill="1" visible="no" active="no"/>
 <layer number="45" name="Holes" color="7" fill="1" visible="no" active="no"/>
-<layer number="46" name="Milling" color="3" fill="1" visible="yes" active="no"/>
-<layer number="47" name="Measures" color="7" fill="1" visible="yes" active="no"/>
-<layer number="48" name="Document" color="7" fill="1" visible="yes" active="no"/>
-<layer number="49" name="Reference" color="7" fill="1" visible="yes" active="no"/>
-<layer number="50" name="dxf" color="7" fill="1" visible="yes" active="no"/>
-<layer number="51" name="tDocu" color="7" fill="1" visible="yes" active="no"/>
-<layer number="52" name="bDocu" color="7" fill="1" visible="yes" active="no"/>
-<layer number="53" name="tGND_GNDA" color="7" fill="9" visible="yes" active="no"/>
-<layer number="54" name="bGND_GNDA" color="1" fill="9" visible="yes" active="no"/>
-<layer number="56" name="wert" color="7" fill="1" visible="yes" active="no"/>
+<layer number="46" name="Milling" color="3" fill="1" visible="no" active="no"/>
+<layer number="47" name="Measures" color="7" fill="1" visible="no" active="no"/>
+<layer number="48" name="Document" color="7" fill="1" visible="no" active="no"/>
+<layer number="49" name="Reference" color="7" fill="1" visible="no" active="no"/>
+<layer number="50" name="dxf" color="7" fill="1" visible="no" active="no"/>
+<layer number="51" name="tDocu" color="7" fill="1" visible="no" active="no"/>
+<layer number="52" name="bDocu" color="7" fill="1" visible="no" active="no"/>
+<layer number="53" name="tGND_GNDA" color="7" fill="9" visible="no" active="no"/>
+<layer number="54" name="bGND_GNDA" color="1" fill="9" visible="no" active="no"/>
+<layer number="56" name="wert" color="7" fill="1" visible="no" active="no"/>
 <layer number="91" name="Nets" color="2" fill="1" visible="yes" active="yes"/>
 <layer number="92" name="Busses" color="1" fill="1" visible="yes" active="yes"/>
@@
 <part name="GND16" library="supply1" deviceset="GND" device=""/>
 <part name="P+10" library="supply1" deviceset="+5V" device=""/>
+<part name="C10" library="SparkFun" deviceset="CAP_POL" device="PTH2" value="4u7"/>
+<part name="GND17" library="supply1" deviceset="GND" device=""/>
 </parts>
 <sheets>
@@
 <text x="254" y="220.98" size="1.778" layer="91">Two slaves boards can be added for 3-axis operation.</text>
 <text x="254" y="215.9" size="1.778" layer="91">Slave boards can use independent ADCs if I2C addresses are different.</text>
-<text x="254" y="205.74" size="1.778" layer="91">Remote board can be used without ADC and feed analogue signal to FLC100 shield.</text>
 <text x="195.58" y="180.34" size="1.778" layer="91">Omit I2C pull-ups on slave boards</text>
 <text x="195.58" y="177.8" size="1.778" layer="91">(Or increase all to 15k - 22k).</text>
@@
 <instance part="GND16" gate="1" x="342.9" y="121.92"/>
 <instance part="P+10" gate="1" x="360.68" y="142.24"/>
+<instance part="C10" gate="G$1" x="327.66" y="129.54"/>
+<instance part="GND17" gate="1" x="327.66" y="121.92"/>
 </instances>
 <busses>
@@
 <pinref part="GND16" gate="1" pin="GND"/>
 <wire x1="342.9" y1="124.46" x2="342.9" y2="127" width="0.1524" layer="91"/>
+</segment>
+<segment>
+<pinref part="C10" gate="G$1" pin="-"/>
+<pinref part="GND17" gate="1" pin="GND"/>
 </segment>
 </net>
@@
 <label x="246.38" y="55.88" size="1.778" layer="95" rot="MR0"/>
 </segment>
-<segment>
-<pinref part="IC3" gate="G$1" pin="VIN"/>
-<wire x1="332.74" y1="134.62" x2="330.2" y2="134.62" width="0.1524" layer="91"/>
-<label x="327.66" y="134.62" size="1.778" layer="95" rot="MR0"/>
-</segment>
 </net>
 <net name="SHDN" class="0">
@@
 </segment>
 </net>
+<net name="VIN_ALT" class="1">
+<segment>
+<pinref part="X1" gate="G$1" pin="2"/>
+<wire x1="251.46" y1="71.12" x2="248.92" y2="71.12" width="0.1524" layer="91"/>
+<label x="246.38" y="71.12" size="1.778" layer="95" rot="MR0"/>
+</segment>
+<segment>
+<pinref part="IC3" gate="G$1" pin="VIN"/>
+<wire x1="332.74" y1="134.62" x2="327.66" y2="134.62" width="0.1524" layer="91"/>
+<label x="322.58" y="134.62" size="1.778" layer="95" rot="MR0"/>
+<junction x="327.66" y="134.62"/>
+<wire x1="327.66" y1="134.62" x2="325.12" y2="134.62" width="0.1524" layer="91"/>
+<pinref part="C10" gate="G$1" pin="+"/>
+<wire x1="327.66" y1="134.62" x2="327.66" y2="132.08" width="0.1524" layer="91"/>
+</segment>
+</net>

Commit message: Adding CAM and Gerber files.
Other:
- note added: "Omit I2C pull-ups on slave boards or increase all to 15k - 22k."
- note added: "One master board required for single-axis operation. Two slaves boards can be added for 3-axis operation. Slave boards can use independent ADCs if I2C addresses are different."
- note removed: "(Or increase all to 15k - 22k)."
- note removed: "Omit I2C pull-ups on slave boards"
- note removed: "One master board required for single-axis operation."
- note removed: "Slave boards can use independent ADCs if I2C addresses are different."
- note removed: "Two slaves boards can be added for 3-axis operation."
Changed lines of the file:
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@@
 <text x="241.3" y="93.98" size="1.778" layer="91">Fit on master board only</text>
 <text x="144.78" y="238.76" size="6.4516" layer="91">FLC100 remote board</text>
-<text x="254" y="226.06" size="1.778" layer="91">One master board required for single-axis operation.</text>
-<text x="254" y="220.98" size="1.778" layer="91">Two slaves boards can be added for 3-axis operation.</text>
-<text x="254" y="215.9" size="1.778" layer="91">Slave boards can use independent ADCs if I2C addresses are different.</text>
-<text x="195.58" y="180.34" size="1.778" layer="91">Omit I2C pull-ups on slave boards</text>
-<text x="195.58" y="177.8" size="1.778" layer="91">(Or increase all to 15k - 22k).</text>
+<text x="254" y="226.06" size="1.778" layer="91" align="top-left">One master board required for single-axis operation.
+Two slaves boards can be added for 3-axis operation.
+Slave boards can use independent ADCs if I2C addresses are different.</text>
+<text x="195.58" y="182.88" size="1.778" layer="91" align="top-left">Omit I2C pull-ups on slave boards
+or increase all to 15k - 22k.</text>
 <text x="307.34" y="40.64" size="2.54" layer="91">Mounting holes</text>
 <text x="45.72" y="25.4" size="2.54" layer="91">Temperature sensor</text>
@@
 <segment>
 <wire x1="172.72" y1="167.64" x2="185.42" y2="167.64" width="0.1524" layer="91"/>
-<label x="170.18" y="167.64" size="1.778" layer="95" rot="MR0"/>
+<label x="195.58" y="167.64" size="1.778" layer="95"/>
 <junction x="185.42" y="167.64"/>
 <wire x1="185.42" y1="167.64" x2="193.04" y2="167.64" width="0.1524" layer="91"/>
@@
 </schematic>
 </drawing>
+<compatibility>
+<note version="6.3" minversion="6.2.2" severity="warning">
+Since Version 6.2.2 text objects can contain more than one line,
+which will not be processed correctly with this version.
+</note>
+</compatibility>
 </eagle>
