File: hardware/FLC100_shield/cloud_detector/cloud_humidity_sensor/cloud_humidity_sensor_v1.sch (EAGLE design)
At the start: 21 parts, among them IC1 HIH613x, IC2 HIH612x, IC3 MLX90614, Q1 2N7000, X1 FLC100 SHIELD, X2 MLX90614

Commit message: Updating boardd and schematic files to match the Gerber files.
Other:
- note added: "1.0"
- note added: "Steve Marple"
Changed lines of the file:
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@@
 7 SDA
 8 +3V3</text>
+<text x="328.168" y="14.478" size="2.54" layer="94">1.0</text>
+<text x="330.708" y="4.318" size="2.54" layer="94">Steve Marple</text>
 </plain>
 <instances>
