File: hardware/FLC100_shield/shield_v2.1/FLC100_shield_v2.1.brd (EAGLE design)
At the start: 99.1 x 53.3 mm, 55 parts, among them IC2 TSR 1-2450, Q1 2N7000, Q2 2N7000, Q3 2N7000, Q4 2N7000, Q5 2N7000, Q6 2N7000, Q7 2N7000, Q8 2N7000, Q9 2N7000, X1 RJ45, X2 RJ11, X3 CLOUD SENSOR, X4 MEGA2560, X5 HUMIDITY

Commit message: Remove unused XRF nets
Connections:
- removed net !XRF_RESET: U$4.5
- removed net RX1: U$4.2@1
- removed net TX1: U$4.3@1
- removed net XRF_ON: U$4.23
- removed net XRF_SLEEP: U$4.7
Changed lines of the file:
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@@
 <via x="69.85" y="13.97" extent="1-16" drill="0.508"/>
-</signal>
-<signal name="XRF_ON">
-<contactref element="U$4" pad="23"/>
 </signal>
 <signal name="!RESET">
@@
 <wire x1="43.942" y1="41.148" x2="56.515" y2="41.148" width="0.254" layer="1"/>
 <wire x1="39.37" y1="45.72" x2="43.942" y2="41.148" width="0.254" layer="1"/>
-</signal>
-<signal name="!XRF_RESET">
-<contactref element="U$4" pad="5"/>
-</signal>
-<signal name="XRF_SLEEP">
-<contactref element="U$4" pad="7"/>
 </signal>
 <signal name="A7">
@@
 <wire x1="28.956" y1="50.8" x2="28.956" y2="47.244" width="0.254" layer="16"/>
 </signal>
-<signal name="RX1">
-<contactref element="U$4" pad="2@1"/>
-</signal>
-<signal name="TX1">
-<contactref element="U$4" pad="3@1"/>
-</signal>
 <signal name="N$10" class="1">
