File: hardware/RPi_Clock_I2C/v1.0.0/RPi_Clock_I2C.brd (EAGLE design)
At the start: 49.5 x 49.5 mm, 31 parts, among them IC1 PCA9517A, IC2 DS1338, IC3 MCP1702-SOT23A, X1 P1, X2 RJ45, X3 RJ11, Y1 32k768

Commit message: Use semantic versioning
Other:
- board text added: "v1.0.0"
- board text removed: "v1.0"
Changed lines of the file:
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@@
 <text x="28.575" y="25.4" size="1.27" layer="25" ratio="10" align="center-right">RTC:</text>
 <rectangle x1="24.13" y1="21.336" x2="35.56" y2="24.384" layer="121"/>
-<text x="34.29" y="36.83" size="1.27" layer="25" ratio="10">v1.0</text>
+<text x="33.02" y="36.83" size="1.27" layer="25" ratio="10">v1.0.0</text>
 <rectangle x1="1.27" y1="1.27" x2="8.128" y2="30.48" layer="121"/>
 <text x="7.62" y="13.97" size="1.016" layer="122" ratio="10" rot="MR270">Steve Marple
