File: hardware/RPi_Clock_I2C/v1.0.0/RPi_Clock_I2C.sch (EAGLE design)
At the start: 31 parts, among them IC1 PCA9517A, IC2 DS1338, IC3 MCP1702-SOT23A, X1 P1, X2 RJ45, X3 RJ11, Y1 32k768

Commit message: Use semantic versioning
Other:
- note added: "1.0"
- note removed: "2.1a"
Changed lines of the file:
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@@
 <text x="-137.16" y="-60.96" size="2.54" layer="91">3V3 regulator</text>
 <text x="158.242" y="-71.882" size="2.54" layer="94">Steve Marple</text>
-<text x="155.702" y="-61.722" size="2.54" layer="94">2.1a</text>
+<text x="155.702" y="-61.722" size="2.54" layer="94">1.0</text>
 <text x="101.6" y="43.18" size="1.778" layer="91">SHUTDOWN held low
 permanently for
